File: electronics/usbc-pcb/usbc.kicad_pcb (KiCad board)
At the start: 2 copper layers, 14 x 13.6 mm, 6 parts, among them J1 USB4736-GF-A, J2 To joystick PCB

Commit message: Add a charge LED beside the V0.24 charging port
Put a red side-looking LED (Lite-On LTST-S270KRKT) on the USB-C PCB,
at its front edge beside the receptacle, with a 1 k resistor and a wire
pad to XIAO D8. The board grows from 14 to 19 mm wide to carry it. The
housing gets a 1.6 mm window through the panel on the LED axis, filled
with clear epoxy, clear of the gasket pocket and the plug overmold.

The charger's CHG signal reaches no XIAO pad, so the firmware copies it
to D8: the LED is on while the cell charges and off otherwise. Specify
the power behaviour: no power switch, A + B + C held 3 s to turn off,
auto-off after 6 h without input, wake on any button or on plugging in
a charger.

Signed-off-by: Marc Cirauqui <marc@tetrate.io>
Parts:
- added D1: Red, orr:LED_LiteOn_LTST-S270, F.Cu at (107.5, 99.1)
- added J3: To XIAO D8, orr:WirePad_1x01, F.Cu at (108.2, 93.0)
- added R3: 1k, Resistor_SMD:R_0603_1608Metric, F.Cu at (108.5, 96.3)
Routing:
- net /LED: track 0.00 -> 2.60 mm
- net /LED_A: track 0.00 -> 1.97 mm
Other:
- board size 14 x 13.6 mm -> 19 x 13.6 mm
- board text added: "LED"
