File: electronics/joystick-pcb/joystick.kicad_pcb (KiCad board)
At the start: 2 copper layers, 20.6 x 22.4 mm, 10 parts, among them J1 Supply in, J2 To XIAO, SW1 KSC222JLFS, SW2 KSC222JLFS, SW3 KSC222JLFS, SW4 KSC222JLFS

Commit message: Switch the joystick to the KSC221JLFS and widen the knob push gap
LCSC has no KSC222JLFS (C221728) in stock. The KSC221JLFS (C221726)
has the same 2 N force, body and J-bend land pattern, so the joystick
PCB layout is unchanged; it has standard silver contacts (500,000
operations instead of 1,000,000) and up to 0.65 mm travel instead of
0.5 mm.

In the V0.24 CAD, the knob push gap grows from 0.7 to 0.9 mm and the
knob from 5.5 to 5.7 mm proud, so every switch trips before the knob
stop. The radial knob insert moves from 2.9 to 3.2 mm below the knob
top, away from the rim underside, where it left a 0.15 mm wall.

Regenerate the joystick PCB, schematic and fabrication files, add the
V0.24 schematic image and update the docs. Note that with nominal
switch travel a hard push loads the switches before the knob stop.

Signed-off-by: Marc Cirauqui <marc@tetrate.io>
Parts:
- SW1, SW2, SW3, SW4: value KSC222JLFS -> KSC221JLFS
