File: electronics/joystick-pcb/joystick.kicad_sch (KiCad schematic)
At the start: 8 parts, among them J1 Supply in, J2 To XIAO, SW1 KSC222JLFS, SW2 KSC222JLFS, SW3 KSC222JLFS, SW4 KSC222JLFS

Commit message: Switch the joystick to the KSC221JLFS and widen the knob push gap
LCSC has no KSC222JLFS (C221728) in stock. The KSC221JLFS (C221726)
has the same 2 N force, body and J-bend land pattern, so the joystick
PCB layout is unchanged; it has standard silver contacts (500,000
operations instead of 1,000,000) and up to 0.65 mm travel instead of
0.5 mm.

In the V0.24 CAD, the knob push gap grows from 0.7 to 0.9 mm and the
knob from 5.5 to 5.7 mm proud, so every switch trips before the knob
stop. The radial knob insert moves from 2.9 to 3.2 mm below the knob
top, away from the rim underside, where it left a 0.15 mm wall.

Regenerate the joystick PCB, schematic and fabrication files, add the
V0.24 schematic image and update the docs. Note that with nominal
switch travel a hard push loads the switches before the knob stop.

Signed-off-by: Marc Cirauqui <marc@tetrate.io>
Parts:
- SW1, SW2, SW3, SW4: value KSC222JLFS -> KSC221JLFS; symbol orr:KSC222JLFS -> orr:KSC221JLFS; LCSC C221728 -> C221726; MPN KSC222JLFS -> KSC221JLFS
Changed lines of the file:
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@@
 (wire (pts (xy 152.40 58.42) (xy 147.32 58.42)) (stroke (width 0) (type default)))
 (label "LEFT" (at 147.32 58.42 180) (effects (font (size 1.27 1.27)) (justify right bottom)))
-(symbol (lib_id "orr:KSC222JLFS") (at 50.80 96.52 0) (unit 1) (exclude_from_sim no) (in_bom yes) (on_board yes) (dnp no) (property "Reference" "SW1" (at 50.80 90.17 0) (effects (font (size 1.27 1.27)))) (property "Value" "KSC222JLFS" (at 50.80 104.14 0) (effects (font (size 1.27 1.27)))) (property "Footprint" "orr:KSC2_SMD_6.2x6.2mm" (at 50.80 96.52 0) (effects (font (size 1.27 1.27)) (hide yes))) (property "Datasheet" "" (at 50.80 96.52 0) (effects (font (size 1.27 1.27)) (hide yes))) (property "Manufacturer" "C&K" (at 50.80 96.52 0) (effects (font (size 1.27 1.27)) (hide yes))) (property "MPN" "KSC222JLFS" (at 50.80 96.52 0) (effects (font (size 1.27 1.27)) (hide yes))) (property "LCSC" "C221728" (at 50.80 96.52 0) (effects (font (size 1.27 1.27)) (hide yes))) (pin "1") (pin "2") (pin "3") (pin "4") (instances (project "joystick" (path "/aeb67614-4432-546e-8581-3a33afebe9cc" (reference "SW1") (unit 1)))))
+(symbol (lib_id "orr:KSC221JLFS") (at 50.80 96.52 0) (unit 1) (exclude_from_sim no) (in_bom yes) (on_board yes) (dnp no) (property "Reference" "SW1" (at 50.80 90.17 0) (effects (font (size 1.27 1.27)))) (property "Value" "KSC221JLFS" (at 50.80 104.14 0) (effects (font (size 1.27 1.27)))) (property "Footprint" "orr:KSC2_SMD_6.2x6.2mm" (at 50.80 96.52 0) (effects (font (size 1.27 1.27)) (hide yes))) (property "Datasheet" "" (at 50.80 96.52 0) (effects (font (size 1.27 1.27)) (hide yes))) (property "Manufacturer" "C&K" (at 50.80 96.52 0) (effects (font (size 1.27 1.27)) (hide yes))) (property "MPN" "KSC221JLFS" (at 50.80 96.52 0) (effects (font (size 1.27 1.27)) (hide yes))) (property "LCSC" "C221726" (at 50.80 96.52 0) (effects (font (size 1.27 1.27)) (hide yes))) (pin "1") (pin "2") (pin "3") (pin "4") (instances (project "joystick" (path "/aeb67614-4432-546e-8581-3a33afebe9cc" (reference "SW1") (unit 1)))))
 (no_connect (at 43.18 95.25))
 (wire (pts (xy 58.42 95.25) (xy 60.96 95.25)) (stroke (width 0) (type default)))
@@
 (label "UP" (at 40.64 100.33 180) (effects (font (size 1.27 1.27)) (justify right bottom)))
 (no_connect (at 58.42 100.33))
-(symbol (lib_id "orr:KSC222JLFS") (at 83.82 96.52 0) (unit 1) (exclude_from_sim no) (in_bom yes) (on_board yes) (dnp no) (property "Reference" "SW2" (at 83.82 90.17 0) (effects (font (size 1.27 1.27)))) (property "Value" "KSC222JLFS" (at 83.82 104.14 0) (effects (font (size 1.27 1.27)))) (property "Footprint" "orr:KSC2_SMD_6.2x6.2mm" (at 83.82 96.52 0) (effects (font (size 1.27 1.27)) (hide yes))) (property "Datasheet" "" (at 83.82 96.52 0) (effects (font (size 1.27 1.27)) (hide yes))) (property "Manufacturer" "C&K" (at 83.82 96.52 0) (effects (font (size 1.27 1.27)) (hide yes))) (property "MPN" "KSC222JLFS" (at 83.82 96.52 0) (effects (font (size 1.27 1.27)) (hide yes))) (property "LCSC" "C221728" (at 83.82 96.52 0) (effects (font (size 1.27 1.27)) (hide yes))) (pin "1") (pin "2") (pin "3") (pin "4") (instances (project "joystick" (path "/aeb67614-4432-546e-8581-3a33afebe9cc" (reference "SW2") (unit 1)))))
+(symbol (lib_id "orr:KSC221JLFS") (at 83.82 96.52 0) (unit 1) (exclude_from_sim no) (in_bom yes) (on_board yes) (dnp no) (property "Reference" "SW2" (at 83.82 90.17 0) (effects (font (size 1.27 1.27)))) (property "Value" "KSC221JLFS" (at 83.82 104.14 0) (effects (font (size 1.27 1.27)))) (property "Footprint" "orr:KSC2_SMD_6.2x6.2mm" (at 83.82 96.52 0) (effects (font (size 1.27 1.27)) (hide yes))) (property "Datasheet" "" (at 83.82 96.52 0) (effects (font (size 1.27 1.27)) (hide yes))) (property "Manufacturer" "C&K" (at 83.82 96.52 0) (effects (font (size 1.27 1.27)) (hide yes))) (property "MPN" "KSC221JLFS" (at 83.82 96.52 0) (effects (font (size 1.27 1.27)) (hide yes))) (property "LCSC" "C221726" (at 83.82 96.52 0) (effects (font (size 1.27 1.27)) (hide yes))) (pin "1") (pin "2") (pin "3") (pin "4") (instances (project "joystick" (path "/aeb67614-4432-546e-8581-3a33afebe9cc" (reference "SW2") (unit 1)))))
 (wire (pts (xy 76.20 95.25) (xy 73.66 95.25)) (stroke (width 0) (type default)))
 (symbol (lib_id "power:GND") (at 73.66 95.25 0) (unit 1) (exclude_from_sim no) (in_bom no) (on_board no) (dnp no) (property "Reference" "#PWR09" (at 73.66 99.06 0) (effects (font (size 1.27 1.27)) (hide yes))) (property "Value" "GND" (at 73.66 100.33 0) (effects (font (size 1.27 1.27)))) (property "Footprint" "" (at 73.66 95.25 0) (effects (font (size 1.27 1.27)) (hide yes))) (property "Datasheet" "" (at 73.66 95.25 0) (effects (font (size 1.27 1.27)) (hide yes))) (pin "1") (instances (project "joystick" (path "/aeb67614-4432-546e-8581-3a33afebe9cc" (reference "#PWR09") (unit 1)))))
@@
 (wire (pts (xy 91.44 100.33) (xy 93.98 100.33)) (stroke (width 0) (type default)))
 (label "DOWN" (at 93.98 100.33 0) (effects (font (size 1.27 1.27)) (justify left bottom)))
-(symbol (lib_id "orr:KSC222JLFS") (at 116.84 96.52 0) (unit 1) (exclude_from_sim no) (in_bom yes) (on_board yes) (dnp no) (property "Reference" "SW3" (at 116.84 90.17 0) (effects (font (size 1.27 1.27)))) (property "Value" "KSC222JLFS" (at 116.84 104.14 0) (effects (font (size 1.27 1.27)))) (property "Footprint" "orr:KSC2_SMD_6.2x6.2mm" (at 116.84 96.52 0) (effects (font (size 1.27 1.27)) (hide yes))) (property "Datasheet" "" (at 116.84 96.52 0) (effects (font (size 1.27 1.27)) (hide yes))) (property "Manufacturer" "C&K" (at 116.84 96.52 0) (effects (font (size 1.27 1.27)) (hide yes))) (property "MPN" "KSC222JLFS" (at 116.84 96.52 0) (effects (font (size 1.27 1.27)) (hide yes))) (property "LCSC" "C221728" (at 116.84 96.52 0) (effects (font (size 1.27 1.27)) (hide yes))) (pin "1") (pin "2") (pin "3") (pin "4") (instances (project "joystick" (path "/aeb67614-4432-546e-8581-3a33afebe9cc" (reference "SW3") (unit 1)))))
+(symbol (lib_id "orr:KSC221JLFS") (at 116.84 96.52 0) (unit 1) (exclude_from_sim no) (in_bom yes) (on_board yes) (dnp no) (property "Reference" "SW3" (at 116.84 90.17 0) (effects (font (size 1.27 1.27)))) (property "Value" "KSC221JLFS" (at 116.84 104.14 0) (effects (font (size 1.27 1.27)))) (property "Footprint" "orr:KSC2_SMD_6.2x6.2mm" (at 116.84 96.52 0) (effects (font (size 1.27 1.27)) (hide yes))) (property "Datasheet" "" (at 116.84 96.52 0) (effects (font (size 1.27 1.27)) (hide yes))) (property "Manufacturer" "C&K" (at 116.84 96.52 0) (effects (font (size 1.27 1.27)) (hide yes))) (property "MPN" "KSC221JLFS" (at 116.84 96.52 0) (effects (font (size 1.27 1.27)) (hide yes))) (property "LCSC" "C221726" (at 116.84 96.52 0) (effects (font (size 1.27 1.27)) (hide yes))) (pin "1") (pin "2") (pin "3") (pin "4") (instances (project "joystick" (path "/aeb67614-4432-546e-8581-3a33afebe9cc" (reference "SW3") (unit 1)))))
 (no_connect (at 109.22 95.25))
 (wire (pts (xy 124.46 95.25) (xy 127.00 95.25)) (stroke (width 0) (type default)))
@@
 (symbol (lib_id "power:GND") (at 106.68 100.33 0) (unit 1) (exclude_from_sim no) (in_bom no) (on_board no) (dnp no) (property "Reference" "#PWR10" (at 106.68 104.14 0) (effects (font (size 1.27 1.27)) (hide yes))) (property "Value" "GND" (at 106.68 105.41 0) (effects (font (size 1.27 1.27)))) (property "Footprint" "" (at 106.68 100.33 0) (effects (font (size 1.27 1.27)) (hide yes))) (property "Datasheet" "" (at 106.68 100.33 0) (effects (font (size 1.27 1.27)) (hide yes))) (pin "1") (instances (project "joystick" (path "/aeb67614-4432-546e-8581-3a33afebe9cc" (reference "#PWR10") (unit 1)))))
 (no_connect (at 124.46 100.33))
-(symbol (lib_id "orr:KSC222JLFS") (at 149.86 96.52 0) (unit 1) (exclude_from_sim no) (in_bom yes) (on_board yes) (dnp no) (property "Reference" "SW4" (at 149.86 90.17 0) (effects (font (size 1.27 1.27)))) (property "Value" "KSC222JLFS" (at 149.86 104.14 0) (effects (font (size 1.27 1.27)))) (property "Footprint" "orr:KSC2_SMD_6.2x6.2mm" (at 149.86 96.52 0) (effects (font (size 1.27 1.27)) (hide yes))) (property "Datasheet" "" (at 149.86 96.52 0) (effects (font (size 1.27 1.27)) (hide yes))) (property "Manufacturer" "C&K" (at 149.86 96.52 0) (effects (font (size 1.27 1.27)) (hide yes))) (property "MPN" "KSC222JLFS" (at 149.86 96.52 0) (effects (font (size 1.27 1.27)) (hide yes))) (property "LCSC" "C221728" (at 149.86 96.52 0) (effects (font (size 1.27 1.27)) (hide yes))) (pin "1") (pin "2") (pin "3") (pin "4") (instances (project "joystick" (path "/aeb67614-4432-546e-8581-3a33afebe9cc" (reference "SW4") (unit 1)))))
+(symbol (lib_id "orr:KSC221JLFS") (at 149.86 96.52 0) (unit 1) (exclude_from_sim no) (in_bom yes) (on_board yes) (dnp no) (property "Reference" "SW4" (at 149.86 90.17 0) (effects (font (size 1.27 1.27)))) (property "Value" "KSC221JLFS" (at 149.86 104.14 0) (effects (font (size 1.27 1.27)))) (property "Footprint" "orr:KSC2_SMD_6.2x6.2mm" (at 149.86 96.52 0) (effects (font (size 1.27 1.27)) (hide yes))) (property "Datasheet" "" (at 149.86 96.52 0) (effects (font (size 1.27 1.27)) (hide yes))) (property "Manufacturer" "C&K" (at 149.86 96.52 0) (effects (font (size 1.27 1.27)) (hide yes))) (property "MPN" "KSC221JLFS" (at 149.86 96.52 0) (effects (font (size 1.27 1.27)) (hide yes))) (property "LCSC" "C221726" (at 149.86 96.52 0) (effects (font (size 1.27 1.27)) (hide yes))) (pin "1") (pin "2") (pin "3") (pin "4") (instances (project "joystick" (path "/aeb67614-4432-546e-8581-3a33afebe9cc" (reference "SW4") (unit 1)))))
 (no_connect (at 142.24 95.25))
 (wire (pts (xy 157.48 95.25) (xy 160.02 95.25)) (stroke (width 0) (type default)))
