File: electronics/control-pcb/control.kicad_pcb (KiCad board)
At the start: 2 copper layers, 21.4 x 49 mm, 27 parts, among them J1 XIAO D0-D6, J2 XIAO 5V-D7, J3 USB-C board, J4 Joystick, J5 Battery, Q1 AO3401A, SW1 KSC221JLFS, SW2 KSC221JLFS, SW3 KSC221JLFS, U1 MCP73831T-2ACI/OT, U2 TPS70933DBVR

Commit message: Complete the V0.26 model with cables and keypad
Model the bought cables and their plugs and route them: joystick to
control board round the joystick board's top edge, USB-C board to the
control board in front of its rib, and the pouch's own lead straight
to a top-entry PH socket, with the pouch fitted protection board up
(27 mm of lead instead of a 76 mm run or an extension). The keypad
keys lose their back nubs so the sheet prints flat; the switches sit
in the plate holes and the upper bosses pass through the board. Board
sockets, the TVS and the fuse move to clear the plugs.

Signed-off-by: Marc Cirauqui <marc@tetrate.io>
Parts:
- H1, H2: value M2 standoff -> M2
- J5: footprint Connector_JST:JST_PH_S2B-PH-SM4-TB_1x02-1MP_P2.00mm_Horizontal -> Connector_JST:JST_PH_B2B-PH-SM4-TB_1x02-1MP_P2.00mm_Vertical
- moved J5 10.4 mm to (95.2, 84.5), turned to 180 degrees
- moved J3 6.57 mm to (103.4, 81.0), turned to 180 degrees
- moved F1 4.46 mm to (96.7, 90.4)
- moved D1 3.30 mm to (97.0, 95.4), turned to 180 degrees
Routing:
- net GND: track 134.9 -> 120.1 mm, vias 1 -> 5
- net +3V3: track 17.5 -> 28.6 mm, vias 0 -> 1
- net /VBUS_IN: track 5.39 -> 13.7 mm
- net /BAT_SYS: track 34.5 -> 26.4 mm, vias 4 -> 0
- net /STAT: track 35.3 -> 43.4 mm
- net /JOY_RIGHT: track 21.7 -> 28.0 mm, vias 1 -> 0
- net /JOY_DOWN: track 22.5 -> 27.9 mm, vias 1 -> 0
- net /VBUS_SENSE: track 16.6 -> 20.8 mm, vias 1 -> 0
- net /BAT: track 25.9 -> 21.7 mm, vias 2 -> 0
- net /JOY_UP: track 22.2 -> 26.0 mm
- net /VBAT_SENSE: track 25.4 -> 27.9 mm
- net /VBUS: track 35.6 -> 34.6 mm, vias 3 -> 2
- net /JOY_LEFT: vias 0 -> 1

Commit message: Mark the battery polarity at J5
"+" and "-" on the control board's rear silkscreen beside J5 let a
builder check a pouch's plug against pin 1 (BAT) before plugging it
in. JST's PH drawing does not settle which side of the plug the latch
is on, so the marks and a meter are the check. The board is routed
again; ERC and DRC show no errors.

Signed-off-by: Marc Cirauqui <marc@tetrate.io>
Other:
- board text added: "+"
- board text added: "-"

Commit message: Apply the control board review fixes
An independent review found no critical defect. R3 and R5 become
150k so D8 and D9 stay under the XIAO's pin limit with a low cell; C3
and C4 become 4.7 uF, above the TPS709's output minimum and the same
part as C1/C2; D1 becomes the 65 uA leakage SMBJ5.0A. The README
records the open points: charge termination with the XIAO's load,
overvoltage above the charger's rating, and a reversed cell with USB
plugged in.

Signed-off-by: Marc Cirauqui <marc@tetrate.io>
Parts:
- C3, C4: value 2.2u -> 4.7u
- R3, R5: value 200k -> 150k
