File: electronics/usbc-pcb-rev-b/usbc.kicad_sch (KiCad schematic)
At the start: 6 parts, among them J1 USB4736-GF-A, J2 To control board

Commit message: Use the in-stock YAGEO 1k for the USB-C board's R3
LCSC has no stock of the UNI-ROYAL 0603WAF1001T5E (C21190); it
would be backordered. The YAGEO RC0603FR-071KL (C22548) is the same
1 kOhm 1 % 100 mW 0603 resistor, with millions in stock. LCSC sells
it in multiples of 100, so the order list asks for 100.

Only the R3 fields change in the schematic and the board; the
Gerbers stay the same, so boards already ordered still apply.

Signed-off-by: Marc Cirauqui <marc@tetrate.io>
Parts:
- R3: LCSC C21190 -> C22548; MPN 0603WAF1001T5E -> RC0603FR-071KL; Manufacturer UNI-ROYAL -> YAGEO
Changed lines of the file:
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@@
 (wire (pts (xy 156.21 38.10) (xy 158.75 38.10)) (stroke (width 0) (type default)))
 (label "LED_A" (at 158.75 38.10 0) (effects (font (size 1.27 1.27)) (justify left bottom)))
-(symbol (lib_id "Device:R") (at 190.50 38.10 0) (unit 1) (exclude_from_sim no) (in_bom yes) (on_board yes) (dnp no) (property "Reference" "R3" (at 190.50 31.75 0) (effects (font (size 1.27 1.27)))) (property "Value" "1k" (at 190.50 45.72 0) (effects (font (size 1.27 1.27)))) (property "Footprint" "Resistor_SMD:R_0603_1608Metric" (at 190.50 38.10 0) (effects (font (size 1.27 1.27)) (hide yes))) (property "Datasheet" "" (at 190.50 38.10 0) (effects (font (size 1.27 1.27)) (hide yes))) (property "MPN" "0603WAF1001T5E" (at 190.50 38.10 0) (effects (font (size 1.27 1.27)) (hide yes))) (property "Manufacturer" "UNI-ROYAL" (at 190.50 38.10 0) (effects (font (size 1.27 1.27)) (hide yes))) (property "LCSC" "C21190" (at 190.50 38.10 0) (effects (font (size 1.27 1.27)) (hide yes))) (pin "1") (pin "2") (instances (project "usbc" (path "/08ce0834-8b21-5094-b645-7be85cd89c12" (reference "R3") (unit 1)))))
+(symbol (lib_id "Device:R") (at 190.50 38.10 0) (unit 1) (exclude_from_sim no) (in_bom yes) (on_board yes) (dnp no) (property "Reference" "R3" (at 190.50 31.75 0) (effects (font (size 1.27 1.27)))) (property "Value" "1k" (at 190.50 45.72 0) (effects (font (size 1.27 1.27)))) (property "Footprint" "Resistor_SMD:R_0603_1608Metric" (at 190.50 38.10 0) (effects (font (size 1.27 1.27)) (hide yes))) (property "Datasheet" "" (at 190.50 38.10 0) (effects (font (size 1.27 1.27)) (hide yes))) (property "MPN" "RC0603FR-071KL" (at 190.50 38.10 0) (effects (font (size 1.27 1.27)) (hide yes))) (property "Manufacturer" "YAGEO" (at 190.50 38.10 0) (effects (font (size 1.27 1.27)) (hide yes))) (property "LCSC" "C22548" (at 190.50 38.10 0) (effects (font (size 1.27 1.27)) (hide yes))) (pin "1") (pin "2") (instances (project "usbc" (path "/08ce0834-8b21-5094-b645-7be85cd89c12" (reference "R3") (unit 1)))))
 (wire (pts (xy 190.50 34.29) (xy 190.50 31.75)) (stroke (width 0) (type default)))
 (label "LED_A" (at 190.50 31.75 0) (effects (font (size 1.27 1.27)) (justify left bottom)))
